Commit message: nearly

File: src_cpp/description/robot.urdf.xacro (robot description, xacro)
@@ -1,19 +1,9 @@
 <?xml version="1.0"?>
 <robot xmlns:xacro="http://www.ros.org/wiki/xacro"  name="dvt_robot">
-    <!-- <xacro:arg name="use_ros2_control"              default="true"/> -->
-    <!-- <xacro:arg name="use_ros2_control_gz_sim"       default="false"/> -->
+    <xacro:arg name="use_ros2_control_gz_sim"       default="false"/>
     <!-- Robot_frames -->
     <xacro:include filename = "robot_core.xacro" />
     <xacro:include filename = "ros2_control.xacro" />
-    <!-- Controls -->
-    <!-- <xacro:if value="$(arg use_ros2_control)">
-        <xacro:include filename = "ros2_control.xacro" />
-    </xacro:if> -->
-    <!-- <xacro:unless value="$(arg use_ros2_control)">
-        <xacro:include filename = "gz_diff_drive_control.xacro" />
-    </xacro:unless> -->
     <!-- Sensors -->
     <xacro:include filename = "lidar.xacro" />
-    <!-- <xacro:include filename = "camera.xacro" /> -->
-    <!-- <xacro:include filename = "depth_camera.xacro" /> -->
 </robot>

File: src_cpp/description/ros2_control.xacro (robot description, xacro)
@@ -1,32 +1,64 @@
 <?xml version="1.0"?>
 <robot xmlns:xacro="http://www.ros.org/wiki/xacro">
-    <ros2_control name="dvt_robot_control" type="system">
-        <hardware>
-            <plugin>gz_ros2_control/GazeboSimSystem</plugin>
-        </hardware>
-        <joint name="left_wheel_joint">
-            <command_interface name="velocity">
-                   <param name="min">-10</param>
-                <param name="max">10</param>
-            </command_interface>
-            <state_interface name="velocity"/>
-            <state_interface name="position"/>
-        </joint>
-        <joint name="right_wheel_joint">
-            <command_interface name="velocity">
-                <param name="min">-10</param>
-                <param name="max">10</param>
-            </command_interface>
-            <state_interface name="velocity"/>
-            <state_interface name="position"/>
-        </joint>
-    </ros2_control>
-    <gazebo>
-        <plugin filename="gz_ros2_control-system"
-            name="gz_ros2_control::GazeboSimROS2ControlPlugin">
-            <parameters>
-                $(find src_cpp)/config/controller_gz_sim.yaml
-            </parameters>
-        </plugin>
-    </gazebo>
+    <xacro:unless value="$(arg use_ros2_control_gz_sim)">
+        <ros2_control name="RobotSystem" type="system">
+            <hardware>
+                <plugin>diffdrive_arduino/DiffDriveArduinoHardware</plugin>
+                    <param name="left_wheel_name">left_wheel_joint</param>
+                    <param name="right_wheel_name">right_wheel_joint</param>
+                    <param name="loop_rate">30</param>
+                    <param name="device">/dev/ttyUSB1</param>
+                    <param name="baud_rate">115200</param>
+                    <param name="timeout_ms">1000</param>
+                    <param name="enc_counts_per_rev">330</param>
+            </hardware>
+            <joint name="left_wheel_joint">
+                <command_interface name="velocity">
+                    <param name="min">-10</param>
+                    <param name="max">10</param>
+                </command_interface>
+                <state_interface name="position"/>
+                <state_interface name="velocity"/>
+            </joint>
+            <joint name="right_wheel_joint">
+                <command_interface name="velocity">
+                    <param name="min">-10</param>
+                    <param name="max">10</param>
+                </command_interface>
+                <state_interface name="position"/>
+                <state_interface name="velocity"/>
+            </joint>
+        </ros2_control>
+    </xacro:unless>
+    <xacro:if value="$(arg use_ros2_control_gz_sim)">
+        <ros2_control name="dvt_robot_control" type="system">
+            <hardware>
+                <plugin>gz_ros2_control/GazeboSimSystem</plugin>
+            </hardware>
+            <joint name="left_wheel_joint">
+                <command_interface name="velocity">
+                    <param name="min">-10</param>
+                    <param name="max">10</param>
+                </command_interface>
+                <state_interface name="velocity"/>
+                <state_interface name="position"/>
+            </joint>
+            <joint name="right_wheel_joint">
+                <command_interface name="velocity">
+                    <param name="min">-10</param>
+                    <param name="max">10</param>
+                </command_interface>
+                <state_interface name="velocity"/>
+                <state_interface name="position"/>
+            </joint>
+        </ros2_control>
+        <gazebo>
+            <plugin filename="gz_ros2_control-system"
+                name="gz_ros2_control::GazeboSimROS2ControlPlugin">
+                <parameters>
+                    $(find src_cpp)/config/controller_gz_sim.yaml
+                </parameters>
+            </plugin>
+        </gazebo>
+    </xacro:if>
 </robot>
